Commit message: add vision based rtabmap launch file and rviz autolaunch

File: model_robot/urdf/model_robot.xacro (robot description, xacro)
@@ -1,6 +1,155 @@
 <?xml version='1.0'?>
 <robot name="model_robot" xmlns:xacro="http://www.ros.org/wiki/xacro">
+  <xacro:include filename="$(find model_robot)/urdf/model_robot.gazebo"/>
   <link name="robot_footprint"></link>
-  <xacro:include filename="$(find model_robot)/urdf/model_robot.gazebo" />
+  <link name='chassis'>
+    <pose>0 0 0.1 0 0 0</pose>
+    <inertial>
+      <mass value="5.0"/>
+      <origin xyz="0.0 0 0" rpy=" 0 0 0"/>
+      <inertia
+          ixx="0.1" ixy="0" ixz="0"
+          iyy="0.1" iyz="0"
+          izz="0.1"
+      />
+    </inertial>
+    <collision name='collision'>
+      <origin xyz="0 0 0" rpy=" 0 0 0"/>
+      <geometry>
+        <cylinder radius="0.2" length="0.1"/>
+      </geometry>
+    </collision>
+    <visual name='chassis_visual'>
+      <origin xyz="0 0 0" rpy=" 0 0 0"/>
+      <geometry>
+        <cylinder radius="0.2" length="0.1"/>
+      </geometry>
+    </visual>
+    <collision name='back_caster_collision'>
+      <origin xyz="-0.15 0 -0.05" rpy=" 0 0 0"/>
+      <geometry>
+        <sphere radius="0.0499"/>
+      </geometry>
+    </collision>
+    <visual name='back_caster_visual'>
+      <origin xyz="-0.15 0 -0.05" rpy=" 0 0 0"/>
+      <geometry>
+        <sphere radius="0.05"/>
+      </geometry>
+    </visual>
+    <collision name='front_caster_collision'>
+      <origin xyz="0.15 0 -0.05" rpy=" 0 0 0"/>
+      <geometry>
+        <sphere radius="0.0499"/>
+      </geometry>
+    </collision>
+    <visual name='front_caster_visual'>
+      <origin xyz="0.15 0 -0.05" rpy=" 0 0 0"/>
+      <geometry>
+        <sphere radius="0.05"/>
+      </geometry>
+    </visual>
+  </link>
+    <link name="left_wheel">
+    <visual>
+      <origin xyz="0.0 0 0" rpy=" 0  1.5707 1.5707"/>
+      <geometry>
+          <cylinder radius="0.1" length="0.05"/>
+      </geometry>
+    </visual>
+  <collision>
+    <origin xyz="0.0 0 0" rpy=" 0  1.5707 1.5707"/>
+    <geometry>
+        <cylinder radius="0.1" length="0.05"/>
+    </geometry>
+  </collision>
+    <inertial>
+      <mass value="5.0"/>
+      <origin xyz="0.0 0 0" rpy=" 0 1.5707 1.5707"/>
+      <inertia
+          ixx="0.1" ixy="0" ixz="0"
+          iyy="0.1" iyz="0"
+          izz="0.1"
+      />
+    </inertial>
+  </link>
+  <link name="right_wheel">
+  <visual>
+    <origin xyz="0.0 0 0" rpy=" 0  1.5707 1.5707"/>
+    <geometry>
+        <cylinder radius="0.1" length="0.05"/>
+    </geometry>
+  </visual>
+  <collision>
+    <origin xyz="0.0 0 0" rpy=" 0  1.5707 1.5707"/>
+    <geometry>
+        <cylinder radius="0.1" length="0.05"/>
+    </geometry>
+  </collision>
+  <inertial>
+      <mass value="5.0"/>
+      <origin xyz="0.0 0 0" rpy=" 0  1.5707 1.5707"/>
+      <inertia
+          ixx="0.1" ixy="0" ixz="0"
+          iyy="0.1" iyz="0"
+          izz="0.1"
+      />
+    </inertial>
+  </link>
+  <link name="camera">
+    <visual>
+      <origin xyz="0.0 0 0" rpy=" 0 0 0"/>
+      <geometry>
+        <sphere radius= "0.05"/>
+      </geometry>
+    </visual>
+  <collision>
+    <origin xyz="0.0 0 0" rpy=" 0 0 0"/>
+    <geometry>
+        <sphere radius= "0.05"/>
+    </geometry>
+  </collision>
+    <inertial>
+      <mass value="0.1"/>
+      <origin xyz="0.05 0.05 0.05" rpy=" 0 0 0"/>
+      <box_inertia m="0.1" x="0.05" y="0.05" z="0.05"/>
+      <inertia
+          ixx="1e-6" ixy="0" ixz="0"
+          iyy="1e-6" iyz="0"
+          izz="1e-6"
+      />
+    </inertial>
+  </link>
+   <joint name="camera_optical_joint" type="fixed">
+    <origin xyz="0 0 0" rpy="-1.5707 0 -1.5707"/>
+    <parent link="camera"/>
+    <child link="camera_link_optical"/>
+  </joint>
+  <link name="camera_link_optical">
+  </link>
+  <link name="hokuyo">
+    <visual>
+      <origin xyz="0.0 0 0" rpy=" 0 0 0"/>
+      <geometry>
+        <mesh filename="package://model_robot/meshes/hokuyo.dae"/>
+      </geometry>
+    </visual>
+  <collision>
+    <origin xyz="0.0 0 0" rpy=" 0 0 0"/>
+    <geometry>
+        <box size="0.1 0.1 0.1"/>
+    </geometry>
+  </collision>
+    <inertial>
+      <mass value="1e-5"/>
+      <origin xyz="0.05 0.05 0.05" rpy=" 0 0 0"/>
+      <inertia
+          ixx="1e-6" ixy="0" ixz="0"
+          iyy="1e-6" iyz="0"
+          izz="1e-6"
+      />
+    </inertial>
+  </link>
+  <!--Joints-->
   <joint name="robot_footprint_joint" type="fixed">
     <origin xyz="0 0 0" rpy="0 0 0" />
@@ -8,146 +157,4 @@
     <child link="chassis" />
   </joint>
-  <link name='chassis'>
-    <pose>0 0 0.1 0 0 0</pose>
-    <inertial>
-      <mass value="15.0"/>
-      <origin xyz="0.0 0 0" rpy=" 0 0 0"/>
-      <inertia
-          ixx="0.1" ixy="0" ixz="0"
-          iyy="0.1" iyz="0"
-          izz="0.1"
-      />
-    </inertial>
-    <collision name='collision'>
-      <origin xyz="0 0 0" rpy=" 0 0 0"/>
-      <geometry>
-        <cylinder radius="0.2" length="0.1"/>
-      </geometry>
-    </collision>
-    <visual name='chassis_visual'>
-      <origin xyz="0 0 0" rpy=" 0 0 0"/>
-      <geometry>
-        <cylinder radius="0.2" length="0.1"/>
-      </geometry>
-    </visual>
-    <collision name='back_caster_collision'>
-      <origin xyz="-0.15 0 -0.05" rpy=" 0 0 0"/>
-      <geometry>
-        <sphere radius="0.0499"/>
-      </geometry>
-    </collision>
-    <visual name='back_caster_visual'>
-      <origin xyz="-0.15 0 -0.05" rpy=" 0 0 0"/>
-      <geometry>
-        <sphere radius="0.05"/>
-      </geometry>
-    </visual>
-    <collision name='front_caster_collision'>
-      <origin xyz="0.15 0 -0.05" rpy=" 0 0 0"/>
-      <geometry>
-        <sphere radius="0.0499"/>
-      </geometry>
-    </collision>
-    <visual name='front_caster_visual'>
-      <origin xyz="0.15 0 -0.05" rpy=" 0 0 0"/>
-      <geometry>
-        <sphere radius="0.05"/>
-      </geometry>
-    </visual>
-  </link>
-    <link name="left_wheel">
-    <visual>
-      <origin xyz="0.0 0 0" rpy=" 0  1.5707 1.5707"/>
-      <geometry>
-          <cylinder radius="0.1" length="0.05"/>
-      </geometry>
-    </visual>
-  <collision>
-    <origin xyz="0.0 0 0" rpy=" 0  1.5707 1.5707"/>
-    <geometry>
-        <cylinder radius="0.1" length="0.05"/>
-    </geometry>
-  </collision>
-    <inertial>
-      <mass value="5.0"/>
-      <origin xyz="0.0 0 0" rpy=" 0 1.5707 1.5707"/>
-      <inertia
-          ixx="0.1" ixy="0" ixz="0"
-          iyy="0.1" iyz="0"
-          izz="0.1"
-      />
-    </inertial>
-  </link>
-  <link name="right_wheel">
-  <visual>
-    <origin xyz="0.0 0 0" rpy=" 0  1.5707 1.5707"/>
-    <geometry>
-        <cylinder radius="0.1" length="0.05"/>
-    </geometry>
-  </visual>
-  <collision>
-    <origin xyz="0.0 0 0" rpy=" 0  1.5707 1.5707"/>
-    <geometry>
-        <cylinder radius="0.1" length="0.05"/>
-    </geometry>
-  </collision>
-  <inertial>
-      <mass value="5.0"/>
-      <origin xyz="0.0 0 0" rpy=" 0  1.5707 1.5707"/>
-      <inertia
-          ixx="0.1" ixy="0" ixz="0"
-          iyy="0.1" iyz="0"
-          izz="0.1"
-      />
-    </inertial>
-  </link>
-  <link name="camera">
-    <visual>
-      <origin xyz="0.0 0 0" rpy=" 0 0 0"/>
-      <geometry>
-        <sphere radius= "0.05"/>
-      </geometry>
-    </visual>
-  <collision>
-    <origin xyz="0.0 0 0" rpy=" 0 0 0"/>
-    <geometry>
-        <sphere radius= "0.05"/>
-    </geometry>
-  </collision>
-    <inertial>
-      <mass value="0.1"/>
-      <origin xyz="0.05 0.05 0.05" rpy=" 0 0 0"/>
-      <box_inertia m="0.1" x="0.05" y="0.05" z="0.05"/>
-      <inertia
-          ixx="1e-6" ixy="0" ixz="0"
-          iyy="1e-6" iyz="0"
-          izz="1e-6"
-      />
-    </inertial>
-  </link>
-  <link name="hokuyo">
-    <visual>
-      <origin xyz="0.0 0 0" rpy=" 0 0 0"/>
-      <geometry>
-        <mesh filename="package://model_robot/meshes/hokuyo.dae"/>
-      </geometry>
-    </visual>
-  <collision>
-    <origin xyz="0.0 0 0" rpy=" 0 0 0"/>
-    <geometry>
-        <box size="0.1 0.1 0.1"/>
-    </geometry>
-  </collision>
-    <inertial>
-      <mass value="1e-5"/>
-      <origin xyz="0.05 0.05 0.05" rpy=" 0 0 0"/>
-      <inertia
-          ixx="1e-6" ixy="0" ixz="0"
-          iyy="1e-6" iyz="0"
-          izz="1e-6"
-      />
-    </inertial>
-  </link>
-  <!--Joints-->
   <joint type="fixed" name="hokuyo_joint">
     <origin xyz="0.15 0 0.09" rpy="0 0 0"/>

Commit message: add velodyne VLP-16 rather than the 2D LiDAR and simulate its pointcloud detection

File: model_robot/urdf/model_robot.xacro (robot description, xacro)
@@ -128,27 +128,17 @@
   <link name="camera_link_optical">
   </link>
-  <link name="hokuyo">
-    <visual>
-      <origin xyz="0.0 0 0" rpy=" 0 0 0"/>
-      <geometry>
-        <mesh filename="package://model_robot/meshes/hokuyo.dae"/>
-      </geometry>
-    </visual>
-  <collision>
-    <origin xyz="0.0 0 0" rpy=" 0 0 0"/>
-    <geometry>
-        <box size="0.1 0.1 0.1"/>
-    </geometry>
-  </collision>
-    <inertial>
-      <mass value="1e-5"/>
-      <origin xyz="0.05 0.05 0.05" rpy=" 0 0 0"/>
-      <inertia
-          ixx="1e-6" ixy="0" ixz="0"
-          iyy="1e-6" iyz="0"
-          izz="1e-6"
-      />
-    </inertial>
-  </link>
+  <link name="lidar">
+      <inertial>
+        <mass value="0.1"/>
+        <origin xyz="0 0 0"/>
+        <inertia ixx="0.1" ixy="0" ixz="0" iyy="0.1" iyz="0" izz="0.1"/>
+      </inertial>
+      <visual>
+        <origin xyz="0 0 -0.0377" />
+        <geometry>
+          <mesh filename="package://velodyne_description/meshes/VLP16_scan.dae" />
+        </geometry>
+      </visual>
+    </link>
   <!--Joints-->
   <joint name="robot_footprint_joint" type="fixed">
@@ -157,7 +147,7 @@
     <child link="chassis" />
   </joint>
-  <joint type="fixed" name="hokuyo_joint">
+  <joint type="fixed" name="lidar_joint">
     <origin xyz="0.15 0 0.09" rpy="0 0 0"/>
-    <child link="hokuyo"/>
+    <child link="lidar"/>
     <parent link="chassis"/>
     <axis xyz="0 1 0" rpy="0 0 0"/>

Commit message: robot motion simulation and ideal unicycle cpp model output

File: model_robot/urdf/model_robot.xacro (robot description, xacro)
@@ -138,4 +138,7 @@
         <geometry>
           <mesh filename="package://velodyne_description/meshes/VLP16_scan.dae" />
+          <!--Could be better for visualization <mesh filename="package://velodyne_description/meshes/VLP16_base_1.dae" />
+          <mesh filename="package://velodyne_description/meshes/VLP16_scan.dae" />
+          <mesh filename="package://velodyne_description/meshes/VLP16_base_2.dae" /> -->
         </geometry>
       </visual>
